File: Arduino_AD2Kit/Experimental_Kit.kicad_pcb (KiCad board)
At the start: 2 copper layers, 69.7 x 77 mm, 15 parts, among them J1 Conn_01x05, J2 AD2, J3 Conn_01x02, J4 Conn_01x02, J5 Conn_01x03, J6 CN7, J7 CN10, J8 AD2, J9 Conn_01x02

Commit message: Add AD2 kit V2 and ATmega328P UNO board projects
- Arduino_AD2Kit: update to V2 (adds decoupling caps/resistors, updated PCB)
- Arduino_UNO_ATmega328P: full UNO-compatible ATmega328P board with PCB
- ATmega328P_Minimal: minimal ATmega328P DIP-28 board schematic
- Ignore .history/ folders

Co-Authored-By: Claude Opus 5.5 <noreply@anthropic.com>
Parts:
- removed J2: AD2, Connector_PinSocket_2.54mm:PinSocket_2x15_P2.54mm_Vertical
- added C1: 100nF, Capacitor_SMD:C_1206_3216Metric, F.Cu at (85.5, 90.2)
- added C2: 10uF, Capacitor_SMD:C_0805_2012Metric, F.Cu at (85.5, 95.2)
- added C3: 100nF, Capacitor_SMD:C_0805_2012Metric, F.Cu at (85.6, 77.5)
- added C4: 10uF, Capacitor_SMD:C_1206_3216Metric, F.Cu at (89.6, 77.5)
- added C5: 100nF, Capacitor_SMD:C_0805_2012Metric, F.Cu at (85.5, 56.6)
- added C6: 10uF, Capacitor_SMD:C_1206_3216Metric, F.Cu at (87.0, 53.6)
- added C7: 100nF, Capacitor_SMD:C_1206_3216Metric, F.Cu at (129.5, 59.5)
- added C8: 10uF, Capacitor_SMD:C_1206_3216Metric, F.Cu at (127.0, 55.5)
- added J10: Conn_02x15_Odd_Even, Connector_PinSocket_2.54mm:PinSocket_2x15_P2.54mm_Horizontal, F.Cu at (94.0, 116.3)
- added R1: 1k, Resistor_SMD:R_0805_2012Metric, F.Cu at (132.3, 112.8)
- added R2: 1k, Resistor_SMD:R_0805_2012Metric, F.Cu at (134.3, 112.8)
- added R3: 1k, Resistor_SMD:R_0805_2012Metric, F.Cu at (129.5, 112.8)
- added R4: 1k, Resistor_SMD:R_0805_2012Metric, F.Cu at (127.0, 112.8)
Routing:
- net GND: track 254.0 -> 297.1 mm, vias 1 -> 3
- net +BATT: track 0.00 -> 13.9 mm
- net Net-(J10-Pin_27): track 0.00 -> 9.96 mm, vias 0 -> 1
- net /Ch2N: track 10.6 -> 2.63 mm
- net /Ch1N: track 10.6 -> 2.63 mm
- net AVDD: track 0.00 -> 7.91 mm
- net AREF: track 39.9 -> 47.0 mm, vias 0 -> 2
- net Net-(J10-Pin_28): track 0.00 -> 6.25 mm
- net Net-(J10-Pin_30): track 0.00 -> 6.25 mm
- net Net-(J10-Pin_29): track 0.00 -> 5.42 mm
- net VIN: track 5.08 -> 8.64 mm
- net /Ch1P: track 10.6 -> 7.93 mm
- net /Ch2P: track 10.6 -> 11.7 mm, vias 0 -> 1
