File: Arduino_AD2Kit/Experimental_Kit.kicad_sch (KiCad schematic)
At the start: 11 parts, among them J1 Conn_01x05, J2 AD2, J3 Conn_01x02, J4 Conn_01x02, J5 Conn_01x03, J6 CN7, J7 CN10, J8 AD2, J9 Conn_01x02

Commit message: Add AD2 kit V2 and ATmega328P UNO board projects
- Arduino_AD2Kit: update to V2 (adds decoupling caps/resistors, updated PCB)
- Arduino_UNO_ATmega328P: full UNO-compatible ATmega328P board with PCB
- ATmega328P_Minimal: minimal ATmega328P DIP-28 board schematic
- Ignore .history/ folders

Co-Authored-By: Claude Opus 5.5 <noreply@anthropic.com>
Parts:
- removed J2: AD2, Connector_PinSocket_2.54mm:PinSocket_2x15_P2.54mm_Horizontal, symbol Connector_Generic:Conn_02x15_Odd_Even
- added C1, C7: 100nF, Capacitor_SMD:C_1206_3216Metric, symbol Device:C
- added C2: 10uF, Capacitor_SMD:C_0805_2012Metric, symbol Device:C
- added C3, C5: 100nF, Capacitor_SMD:C_0805_2012Metric, symbol Device:C
- added C4, C6, C8: 10uF, Capacitor_SMD:C_1206_3216Metric, symbol Device:C
- added J10: Conn_02x15_Odd_Even, Connector_PinSocket_2.54mm:PinSocket_2x15_P2.54mm_Horizontal, symbol Connector_Generic:Conn_02x15_Odd_Even
- added R1, R2, R3, R4: 1k, Resistor_SMD:R_0805_2012Metric, symbol Device:R
Connections:
- net +BATT: now also C1.1, C2.1
- net AREF: now also C7.1, C8.1
- net AVDD: now also C5.1, C6.1
- net Ch1N: now also R3.1
- net Ch1P: now also R1.1
- net Ch2N: now also R4.1
- net Ch2P: now also R2.1
- net DIO0: now also J10.15 (Pin_15)
- net DIO1: now also J10.13 (Pin_13)
- net DIO10: now also J10.12 (Pin_12)
- net DIO11: now also J10.10 (Pin_10)
- net DIO12: now also J10.8 (Pin_8)
- net DIO13: now also J10.6 (Pin_6)
- net DIO2: now also J10.11 (Pin_11)
- net DIO3: now also J10.9 (Pin_9)
- net DIO4: now also J10.7 (Pin_7)
- net DIO5: now also J10.5 (Pin_5)
- net DIO6: now also J10.3 (Pin_3)
- net DIO7: now also J10.1 (Pin_1)
- net DIO8: now also J10.16 (Pin_16)
- net DIO9: now also J10.14 (Pin_14)
- net GND: now also C1.2, C2.2, C3.2, C4.2, C5.2, C6.2, C7.2, C8.2, J10.19 (Pin_19), J10.20 (Pin_20), J10.25 (Pin_25), J10.26 (Pin_26)
- net SCL/A5: now also J10.2 (Pin_2)
- net SDA/A4: now also J10.4 (Pin_4)
- net TI: now also J10.17 (Pin_17)
- net TO: now also J10.18 (Pin_18)
- net VIN: now also C3.1, C4.1
- net Vn: now also J10.24 (Pin_24)
- net Vp: now also J10.23 (Pin_23)
- net W1: now also J10.21 (Pin_21)
- net W2: now also J10.22 (Pin_22)
- new net: J10.29 (Pin_29), R1.2
- new net: J10.27 (Pin_27), R2.2
- new net: J10.28 (Pin_28), R4.2
- new net: J10.30 (Pin_30), R3.2
Other:
- moved on the sheet: A1
